Commit message: Surface URDF visual asset readiness

File: examples/noetix-e1/model/robot.urdf (robot description, URDF)
Before this commit: robot noetix_e1_lab_01, 25 links, 24 joints
Links:
- link base_link: geometry visual mesh filename=meshes/base.obj scale=1 1 1
- link chest_link: geometry visual box size=0.28 0.34 0.18
- link left_arm_1: geometry visual cylinder length=0.12 radius=0.035
- link left_leg_1: geometry visual cylinder length=0.14 radius=0.045
- link right_arm_1: geometry visual cylinder length=0.12 radius=0.035
- link torso_link: geometry visual box size=0.22 0.16 0.18
